File: PCBLayout/popperpump/popperPump/popperPump.kicad_sch (KiCad schematic)
At the start: 14 parts, among them M5StackHeader1 M5StackGPIO

Commit message: 2 Fixes
 - Fix the PCB layout, one of the pins was placed wrong :facepalm:

- Remove the timing limits (coming later)

- Update GPIO pin layout for buttons, because I'm dumb
Connections:
- net at DRV8871.1 (Pin_1): no longer M5StackHeader1.22 (Pin_22)
- net at DRV8871.2 (Pin_2): no longer M5StackHeader1.21 (Pin_21)
- net at DRV8871.3 (Pin_3): now also M5StackHeader1.22 (Pin_22)
- net at DRV8871.4 (Pin_4): now also M5StackHeader1.21 (Pin_21)
- net at ButCNeutral1.1, ButCPullDown1.2: now also M5StackHeader1.7 (Pin_7); no longer M5StackHeader1.11 (Pin_11)
